Commit message: Fix 48DoFs model joint constraints

File: templates/XSensModelStyle_48URDFtemplate.urdf (robot description, URDF)
Before this commit: robot XSensStyleModel_template, 49 links, 48 joints
Joints:
- joint jLeftAnkle_rotx: limit lower=-0.610865 upper=0.785398 effort=30 velocity=1.0 -> lower=-0.785398 upper=0.610865 effort=30 velocity=1.0
- joint jRightC7Shoulder_rotx: limit lower=-0.0872665 upper=0.785398 effort=30 velocity=1.0 -> lower=-0.785398 upper=0.0872665 effort=30 velocity=1.0
- joint jRightHip_rotx: limit lower=-0.523599 upper=0.785398 effort=30 velocity=1.0 -> lower=-0.785398 upper=0.523599 effort=30 velocity=1.0
