Commit message: Added rotz joint for Thumb1

File: templates/XSensModelStyle_48URDFhands_template.urdf (robot description, URDF)
Before this commit: robot XSensStyleModel_template_hands, 79 links, 78 joints
Links:
- added link LeftThumb2_f1, mass FAKEMASS
- added link RightThumb2_f1, mass FAKEMASS
Joints:
- added joint jLeftThumb1_rotz: type revolute, parent LeftThumb1, child LeftThumb2_f1, origin xyz=0 0 0 rpy=0 0 0, axis 0 0 1, limit lower=-1.5708 upper=1.48353 effort=30 velocity=1.0
- added joint jRightThumb1_rotz: type revolute, parent RightThumb1, child RightThumb2_f1, origin xyz=0 0 0 rpy=0 0 0, axis 0 0 1, limit lower=-1.5708 upper=1.48353 effort=30 velocity=1.0
- joint jLeftThumb2_rotx: parent LeftThumb1 -> LeftThumb2_f1
- joint jRightThumb2_rotx: parent RightThumb1 -> RightThumb2_f1

Commit message: Added abduction range of motion for the first digits in the model hand template

File: templates/XSensModelStyle_48URDFhands_template.urdf (robot description, URDF)
Before this commit: robot XSensStyleModel_template_hands, 81 links, 80 joints
Links:
- added link LeftIndex2_f1, mass FAKEMASS
- added link LeftMiddle2_f1, mass FAKEMASS
- added link LeftPinky2_f1, mass FAKEMASS
- added link LeftRing2_f1, mass FAKEMASS
- added link RightIndex2_f1, mass FAKEMASS
- added link RightMiddle2_f1, mass FAKEMASS
- added link RightPinky2_f1, mass FAKEMASS
- added link RightRing2_f1, mass FAKEMASS
Joints:
- added joint jLeftIndex1_rotz: type revolute, parent LeftIndex1, child LeftIndex2_f1, origin xyz=0 0 0 rpy=0 0 0, axis 0 0 1, limit lower=-10 upper=10 effort=30 velocity=1.0
- added joint jLeftMiddle1_rotz: type revolute, parent LeftMiddle1, child LeftMiddle2_f1, origin xyz=0 0 0 rpy=0 0 0, axis 0 0 1, limit lower=-10 upper=10 effort=30 velocity=1.0
- added joint jLeftPinky1_rotz: type revolute, parent LeftPinky1, child LeftPinky2_f1, origin xyz=0 0 0 rpy=0 0 0, axis 0 0 1, limit lower=-10 upper=10 effort=30 velocity=1.0
- added joint jLeftRing1_rotz: type revolute, parent LeftRing1, child LeftRing2_f1, origin xyz=0 0 0 rpy=0 0 0, axis 0 0 1, limit lower=-10 upper=10 effort=30 velocity=1.0
- added joint jRightIndex1_rotz: type revolute, parent RightIndex1, child RightIndex2_f1, origin xyz=0 0 0 rpy=0 0 0, axis 0 0 1, limit lower=-10 upper=10 effort=30 velocity=1.0
- added joint jRightMiddle1_rotz: type revolute, parent RightMiddle1, child RightMiddle2_f1, origin xyz=0 0 0 rpy=0 0 0, axis 0 0 1, limit lower=-10 upper=10 effort=30 velocity=1.0
- added joint jRightPinky1_rotz: type revolute, parent RightPinky1, child RightPinky2_f1, origin xyz=0 0 0 rpy=0 0 0, axis 0 0 1, limit lower=-10 upper=10 effort=30 velocity=1.0
- added joint jRightRing1_rotz: type revolute, parent RightRing1, child RightRing2_f1, origin xyz=0 0 0 rpy=0 0 0, axis 0 0 1, limit lower=-10 upper=10 effort=30 velocity=1.0
- joint jLeftIndex2_rotx: parent LeftIndex1 -> LeftIndex2_f1
- joint jLeftMiddle2_rotx: parent LeftMiddle1 -> LeftMiddle2_f1
- joint jLeftPinky2_rotx: parent LeftPinky1 -> LeftPinky2_f1
- joint jLeftRing2_rotx: parent LeftRing1 -> LeftRing2_f1
- joint jRightIndex2_rotx: parent RightIndex1 -> RightIndex2_f1
- joint jRightMiddle2_rotx: parent RightMiddle1 -> RightMiddle2_f1
- joint jRightPinky2_rotx: parent RightPinky1 -> RightPinky2_f1
- joint jRightRing2_rotx: parent RightRing1 -> RightRing2_f1

Commit message: Split palm link into two sublinks to allow hand palm curvature

File: templates/XSensModelStyle_48URDFhands_template.urdf (robot description, URDF)
Before this commit: robot XSensStyleModel_template_hands, 89 links, 88 joints
Links:
- removed link LeftPalm
- removed link RightPalm
- added link LeftPalmCloseToThumb, mass LEFTPALMCLOSETOTHUMBMASS; collision box size=LEFTPALMCLOSETOTHUMB_BOX_SIZE; visual box size=LEFTPALMCLOSETOTHUMB_BOX_SIZE
- added link LeftPalmFarFromThumb, mass LEFTPALMFARFROMTHUMBMASS; collision box size=LEFTPALMFARFROMTHUMB_BOX_SIZE; visual box size=LEFTPALMFARFROMTHUMB_BOX_SIZE
- added link RightPalmCloseToThumb, mass RIGHTPALMCLOSETOTHUMBMASS; collision box size=RIGHTPALMCLOSETOTHUMB_BOX_SIZE; visual box size=RIGHTPALMCLOSETOTHUMB_BOX_SIZE
- added link RightPalmFarFromThumb, mass RIGHTPALMFARFROMTHUMBMASS; collision box size=RIGHTPALMFARFROMTHUMB_BOX_SIZE; visual box size=RIGHTPALMFARFROMTHUMB_BOX_SIZE
Joints:
- added joint jLeftPalm_roty: type revolute, parent LeftPalmCloseToThumb, child LeftPalmFarFromThumb, origin xyz=jLeftPalm_ORIGIN rpy=0 0 0, axis 0 1 0, limit lower=-10 upper=10 effort=30 velocity=1.0
- added joint jRightPalm_roty: type revolute, parent RightPalmCloseToThumb, child RightPalmFarFromThumb, origin xyz=jRightPalm_ORIGIN rpy=0 0 0, axis 0 1 0, limit lower=-10 upper=10 effort=30 velocity=1.0
- joint jLeftIndex1_rotx: parent LeftPalm -> LeftPalmCloseToThumb
- joint jLeftMiddle1_rotx: parent LeftPalm -> LeftPalmCloseToThumb
- joint jLeftPinky1_rotx: parent LeftPalm -> LeftPalmFarFromThumb
- joint jLeftRing1_rotx: parent LeftPalm -> LeftPalmFarFromThumb
- joint jLeftThumb1_roty: parent LeftPalm -> LeftPalmCloseToThumb
- joint jLeftWrist_rotz: child LeftPalm -> LeftPalmCloseToThumb
- joint jRightIndex1_rotx: parent RightPalm -> RightPalmCloseToThumb
- joint jRightMiddle1_rotx: parent RightPalm -> RightPalmCloseToThumb
- joint jRightPinky1_rotx: parent RightPalm -> RightPalmFarFromThumb
- joint jRightRing1_rotx: parent RightPalm -> RightPalmFarFromThumb
- joint jRightThumb1_roty: parent RightPalm -> RightPalmCloseToThumb
- joint jRightWrist_rotz: child RightPalm -> RightPalmCloseToThumb

Commit message: Added marker-driven hand model.
- Added new URDF template.
- Changed dialog boxes.
- Updated README.

File: templates/XSensModelStyle_48URDFhands_template.urdf (robot description, URDF)
Before this commit: robot XSensStyleModel_template_hands, 91 links, 90 joints
Joints:
- joint jRightAnkle_rotx: limit lower=-0.610865 upper=0.785398 effort=30 velocity=1.0 -> lower=-0.785398 upper=0.610865 effort=30 velocity=1.0
- joint jRightC7Shoulder_rotx: limit lower=-0.0872665 upper=0.785398 effort=30 velocity=1.0 -> lower=-0.785398 upper=0.0872665 effort=30 velocity=1.0
- joint jRightHip_rotx: limit lower=-0.523599 upper=0.785398 effort=30 velocity=1.0 -> lower=-0.785398 upper=0.523599 effort=30 velocity=1.0

File: templates/XSensModelStyle_66URDFtemplate.urdf (robot description, URDF)
Before this commit: robot XSensStyleModel_template, 67 links, 66 joints
Joints:
- joint jC1Head_rotx: limit lower=-10.0 upper=10.0 effort=30 velocity=1.0 -> lower=-0.610865 upper=0.610865 effort=30 velocity=1.0
- joint jC1Head_roty: limit lower=-10.0 upper=10.0 effort=30 velocity=1.0 -> lower=-0.436332 upper=0.174533 effort=30 velocity=1.0
- joint jL1T12_rotx: limit lower=-10.0 upper=10.0 effort=30 velocity=1.0 -> lower=-0.610865 upper=0.610865 effort=30 velocity=1.0
- joint jL1T12_roty: limit lower=-10.0 upper=10.0 effort=30 velocity=1.0 -> lower=-0.523599 upper=1.309 effort=30 velocity=1.0
- joint jL4L3_rotx: limit lower=-10.0 upper=10.0 effort=30 velocity=1.0 -> lower=-0.610865 upper=0.610865 effort=30 velocity=1.0
- joint jL4L3_roty: limit lower=-10.0 upper=10.0 effort=30 velocity=1.0 -> lower=-0.523599 upper=1.309 effort=30 velocity=1.0
- joint jL5S1_rotx: limit lower=-10.0 upper=10.0 effort=30 velocity=1.0 -> lower=-0.610865 upper=0.610865 effort=30 velocity=1.0
- joint jL5S1_roty: limit lower=-10.0 upper=10.0 effort=30 velocity=1.0 -> lower=-0.523599 upper=1.309 effort=30 velocity=1.0
- joint jLeftAnkle_rotx: limit lower=-10.0 upper=10.0 effort=30 velocity=1.0 -> lower=-0.785398 upper=0.610865 effort=30 velocity=1.0
- joint jLeftAnkle_roty: limit lower=-10.0 upper=10.0 effort=30 velocity=1.0 -> lower=-0.523599 upper=0.872665 effort=30 velocity=1.0
- joint jLeftAnkle_rotz: limit lower=-10.0 upper=10.0 effort=30 velocity=1.0 -> lower=-0.872665 upper=0.436332 effort=30 velocity=1.0
- joint jLeftBallFoot_roty: limit lower=-10.0 upper=10.0 effort=30 velocity=1.0 -> lower=-0.174533 upper=1.5708 effort=30 velocity=1.0
- joint jLeftC7Shoulder_rotx: limit lower=-10.0 upper=10.0 effort=30 velocity=1.0 -> lower=-0.0872665 upper=0.785398 effort=30 velocity=1.0
- joint jLeftElbow_roty: limit lower=-10.0 upper=10.0 effort=30 velocity=1.0 -> lower=-1.5708 upper=1.48353 effort=30 velocity=1.0
- joint jLeftElbow_rotz: limit lower=-10.0 upper=10.0 effort=30 velocity=1.0 -> lower=-2.53073 upper=0 effort=30 velocity=1.0
- joint jLeftHip_rotx: limit lower=-10.0 upper=10.0 effort=30 velocity=1.0 -> lower=-0.523599 upper=0.785398 effort=30 velocity=1.0
- joint jLeftHip_roty: limit lower=-10.0 upper=10.0 effort=30 velocity=1.0 -> lower=-0.261799 upper=2.0944 effort=30 velocity=1.0
- joint jLeftHip_rotz: limit lower=-10.0 upper=10.0 effort=30 velocity=1.0 -> lower=-0.785398 upper=0.785398 effort=30 velocity=1.0
- joint jLeftKnee_roty: limit lower=-10.0 upper=10.0 effort=30 velocity=1.0 -> lower=0 upper=2.35619 effort=30 velocity=1.0
- joint jLeftKnee_rotz: limit lower=-10.0 upper=10.0 effort=30 velocity=1.0 -> lower=-0.523599 upper=0.698132 effort=30 velocity=1.0
- joint jLeftShoulder_rotx: limit lower=-10.0 upper=10.0 effort=30 velocity=1.0 -> lower=-1.5708 upper=2.35619 effort=30 velocity=1.0
- joint jLeftShoulder_roty: limit lower=-10.0 upper=10.0 effort=30 velocity=1.0 -> lower=-1.5708 upper=1.5708 effort=30 velocity=1.0
- joint jLeftShoulder_rotz: limit lower=-10.0 upper=10.0 effort=30 velocity=1.0 -> lower=-3.14159 upper=0.785398 effort=30 velocity=1.0
- joint jLeftWrist_rotx: limit lower=-10.0 upper=10.0 effort=30 velocity=1.0 -> lower=-1.0472 upper=0.872665 effort=30 velocity=1.0
- joint jLeftWrist_rotz: limit lower=-10.0 upper=10.0 effort=30 velocity=1.0 -> lower=-0.349066 upper=0.523599 effort=30 velocity=1.0
- joint jRightAnkle_rotx: limit lower=-10.0 upper=10.0 effort=30 velocity=1.0 -> lower=-0.610865 upper=0.785398 effort=30 velocity=1.0
- joint jRightAnkle_roty: limit lower=-10.0 upper=10.0 effort=30 velocity=1.0 -> lower=-0.523599 upper=0.872665 effort=30 velocity=1.0
- joint jRightAnkle_rotz: limit lower=-10.0 upper=10.0 effort=30 velocity=1.0 -> lower=-0.436332 upper=0.872665 effort=30 velocity=1.0
- joint jRightBallFoot_roty: limit lower=-10.0 upper=10.0 effort=30 velocity=1.0 -> lower=-0.174533 upper=1.5708 effort=30 velocity=1.0
- joint jRightC7Shoulder_rotx: limit lower=-10.0 upper=10.0 effort=30 velocity=1.0 -> lower=-0.785398 upper=0.0872665 effort=30 velocity=1.0
- joint jRightElbow_roty: limit lower=-10.0 upper=10.0 effort=30 velocity=1.0 -> lower=-1.5708 upper=1.48353 effort=30 velocity=1.0
- joint jRightElbow_rotz: limit lower=-10.0 upper=10.0 effort=30 velocity=1.0 -> lower=0 upper=2.53073 effort=30 velocity=1.0
- joint jRightHip_rotx: limit lower=-10.0 upper=10.0 effort=30 velocity=1.0 -> lower=-0.785398 upper=0.523599 effort=30 velocity=1.0
- joint jRightHip_roty: limit lower=-10.0 upper=10.0 effort=30 velocity=1.0 -> lower=-0.261799 upper=2.0944 effort=30 velocity=1.0
- joint jRightHip_rotz: limit lower=-10.0 upper=10.0 effort=30 velocity=1.0 -> lower=-0.785398 upper=0.785398 effort=30 velocity=1.0
- joint jRightKnee_roty: limit lower=-10.0 upper=10.0 effort=30 velocity=1.0 -> lower=0 upper=2.35619 effort=30 velocity=1.0
- joint jRightKnee_rotz: limit lower=-10.0 upper=10.0 effort=30 velocity=1.0 -> lower=-0.698132 upper=0.523599 effort=30 velocity=1.0
- joint jRightShoulder_rotx: limit lower=-10.0 upper=10.0 effort=30 velocity=1.0 -> lower=-2.35619 upper=1.5708 effort=30 velocity=1.0
- joint jRightShoulder_roty: limit lower=-10.0 upper=10.0 effort=30 velocity=1.0 -> lower=-1.5708 upper=1.5708 effort=30 velocity=1.0
- joint jRightShoulder_rotz: limit lower=-10.0 upper=10.0 effort=30 velocity=1.0 -> lower=-0.785398 upper=3.14159 effort=30 velocity=1.0
- joint jRightWrist_rotx: limit lower=-10.0 upper=10.0 effort=30 velocity=1.0 -> lower=-0.872665 upper=1.0472 effort=30 velocity=1.0
- joint jRightWrist_rotz: limit lower=-10.0 upper=10.0 effort=30 velocity=1.0 -> lower=-0.523599 upper=0.349066 effort=30 velocity=1.0
- joint jT1C7_rotx: limit lower=-10.0 upper=10.0 effort=30 velocity=1.0 -> lower=-0.610865 upper=0.610865 effort=30 velocity=1.0
- joint jT1C7_roty: limit lower=-10.0 upper=10.0 effort=30 velocity=1.0 -> lower=-0.959931 upper=1.5708 effort=30 velocity=1.0
- joint jT1C7_rotz: limit lower=-10.0 upper=10.0 effort=30 velocity=1.0 -> lower=-1.22173 upper=1.22173 effort=30 velocity=1.0
- joint jT9T8_rotx: limit lower=-10.0 upper=10.0 effort=30 velocity=1.0 -> lower=-0.349066 upper=0.349066 effort=30 velocity=1.0
- joint jT9T8_roty: limit lower=-10.0 upper=10.0 effort=30 velocity=1.0 -> lower=-0.261799 upper=0.698132 effort=30 velocity=1.0
- joint jT9T8_rotz: limit lower=-10.0 upper=10.0 effort=30 velocity=1.0 -> lower=-0.610865 upper=0.610865 effort=30 velocity=1.0
